File: orbi_projetos/schemas/orbi/orbi.kicad_sch (KiCad schematic)
At the start: 24 parts, among them J1 USB_C_Receptacle_USB2.0_16P, SW1 SW_Push, SW2 SW_Push, U1 MPU-6050, U2 ESP32-S2, U3 BMP280, U4 RXM-GPS-FM, U5 TLV75801PDRV, U6 D3V3XA4B10LP

Commit message: Inserindo componentes de display
Parts:
- added U7, U8: EA_DOGS104B-A, Display:EA_DOGS104X-A, symbol Display_Graphic:EA_DOGS104B-A
Changed lines of the file:
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@@
+	)
+	(symbol
+		(lib_id "Display_Graphic:EA_DOGS104B-A")
+		(at 69.85 172.72 0)
+		(unit 1)
+		(exclude_from_sim no)
+		(in_bom yes)
+		(on_board yes)
+		(dnp no)
+		(fields_autoplaced yes)
+		(property "Reference" "U8"
+			(at 71.9933 157.48 0)
+			(effects
+				(font
+					(size 1.27 1.27)
+				)
+				(justify left)
+			)
+		)
+		(property "Value" "EA_DOGS104B-A"
+			(at 71.9933 160.02 0)
+			(effects
+				(font
+					(size 1.27 1.27)
+				)
+				(justify left)
+			)
+		)
+		(property "Footprint" "Display:EA_DOGS104X-A"
+			(at 69.85 187.96 0)
+			(effects
+				(font
+					(size 1.27 1.27)
+				)
+				(hide yes)
+			)
+		)
+		(property "Datasheet" "http://www.lcd-module.com/fileadmin/eng/pdf/doma/dogs104e.pdf"
+			(at 80.01 180.34 0)
+			(effects
+				(font
+					(size 1.27 1.27)
+				)
+				(hide yes)
+			)
+		)
+		(property "Description" "LCD 4x10 character display blue transmissive background, +3.3V VDD, I2C or SPI"
+			(at 69.85 172.72 0)
+			(effects
+				(font
+					(size 1.27 1.27)
+				)
+				(hide yes)
+			)
+		)
+		(pin "10"
+		)
+		(pin "2"
+		)
+		(pin "14"
+		)
+		(pin "19"
+		)
+		(pin "13"
+		)
+		(pin "15"
+		)
+		(pin "1"
+		)
+		(pin "17"
+		)
+		(pin "9"
+		)
+		(pin "20"
+		)
+		(pin "16"
+		)
+		(pin "11"
+		)
+		(pin "12"
+		)
+		(pin "18"
+		)
+		(instances
+			(project ""
+				(path "/cc5c0dcb-4b74-462c-86de-ed43f1f5f7f0"
+					(reference "U8")
+					(unit 1)
+				)
+			)
+		)
 	)
 	(symbol
@@
 					(unit 1)
 				)
+			)
+		)
+	)
+	(symbol
+		(lib_id "Display_Graphic:EA_DOGS104B-A")
+		(at 93.98 139.7 0)
+		(unit 1)
+		(exclude_from_sim no)
+		(in_bom yes)
+		(on_board yes)
+		(dnp no)
+		(fields_autoplaced yes)
+		(property "Reference" "U7"
+			(at 96.1233 124.46 0)
+			(effects
+				(font
+					(size 1.27 1.27)
+				)
+				(justify left)
+			)
+		)
+		(property "Value" "EA_DOGS104B-A"
+			(at 96.1233 127 0)
+			(effects
+				(font
+					(size 1.27 1.27)
+				)
+				(justify left)
+			)
+		)
+		(property "Footprint" "Display:EA_DOGS104X-A"
+			(at 93.98 154.94 0)
+			(effects
+				(font
+					(size 1.27 1.27)
+				)
+				(hide yes)
+			)
+		)
+		(property "Datasheet" "http://www.lcd-module.com/fileadmin/eng/pdf/doma/dogs104e.pdf"
+			(at 104.14 147.32 0)
+			(effects
+				(font
+					(size 1.27 1.27)
+				)
+				(hide yes)
+			)
+		)
+		(property "Description" "LCD 4x10 character display blue transmissive background, +3.3V VDD, I2C or SPI"
+			(at 93.98 139.7 0)
+			(effects
+				(font
+					(size 1.27 1.27)
+				)
+				(hide yes)
+			)
+		)
+		(pin "10"
+		)
+		(pin "2"
+		)
+		(pin "14"
+		)
+		(pin "19"
+		)
+		(pin "13"
+		)
+		(pin "15"
+		)
+		(pin "1"
+		)
+		(pin "17"
+		)
+		(pin "9"
+		)
+		(pin "20"
+		)
+		(pin "16"
+		)
+		(pin "11"
+		)
+		(pin "12"
+		)
+		(pin "18"
+		)
+		(instances
+			(project ""
+				(path "/cc5c0dcb-4b74-462c-86de-ed43f1f5f7f0"
+					(reference "U7")
+					(unit 1)
+				)

Commit message: Adição de mais alguns componentes
Parts:
- added SW3, SW4, SW5, SW6: SW_Push, symbol Switch:SW_Push
Other:
- moved on the sheet: SW1, SW2
